File: Tiny85DevBoard.kicad_pcb (KiCad board)
At the start: 2 copper layers, 29.2 x 40.6 mm, 13 parts, among them J1 Screw_Terminal_01x02, J2 AVR-ISP-6, J3 Conn_01x04_Female, J4 Conn_01x04_Female, SW1 SW_SPDT, SW2 Reset, U1 LD1117S33TR_SOT223, U2 ATtiny85-20PU

Commit message: Added a board name to the silkscreen.
Other:
- board text added: "Tiny85 Dev Board"
Changed lines of the file:
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@@
   (general
     (thickness 1.6)
-    (drawings 16)
+    (drawings 17)
     (tracks 64)
     (zones 0)
@@
     (visible_elements FFFFFF7F)
     (pcbplotparams
-      (layerselection 0x01000_fffffffe)
+      (layerselection 0x010f0_ffffffff)
       (usegerberextensions false)
       (usegerberattributes false)
@@
       (padsonsilk false)
       (subtractmaskfromsilk false)
-      (outputformat 5)
+      (outputformat 1)
       (mirror false)
       (drillshape 0)
@@
     )
   )
+  (gr_text "Tiny85 Dev Board" (at 170.18 127) (layer F.SilkS)
+    (effects (font (size 1 1) (thickness 0.2)))
+  )
   (gr_text ISP (at 184.404 124.968) (layer F.SilkS)
